Commit message: Update ROBOT_2.urdf

File: ROBOT_2/ROBOT_2.urdf (robot description, URDF)
Before this commit: robot ROBOT, 8 links, 7 joints
Joints:
- joint End_Link_Revolute-7: child Link6 -> End_Link; parent End_Link -> Link6
- joint LInk2_Revolute-2: child Link1 -> LInk2; parent LInk2 -> Link1
- joint Link3_Revolute-3: child LInk2 -> Link3; parent Link3 -> LInk2
- joint Link4_Revolute-4: child Link3 -> Link4; parent Link4 -> Link3
- joint Link6_Revolute-6: child Link5 -> Link6; parent Link6 -> Link5
